File: src/assets/files/projects/p2-first-board/P2PlugTestUSB.sch (EAGLE design)
At the start: 24 parts, among them U1 TPS62026

Commit message: P2 First Board update
Changed lines of the file:
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@@
 <part name="U$5" library="rickk2" deviceset="SWITCH-PTS645" device=""/>
 <part name="GND11" library="rickk2" deviceset="GND" device=""/>
-<part name="SUPPLY4" library="rickk2" deviceset="3V3" device=""/>
 <part name="SUPPLY1" library="rickk2" deviceset="3V3" device=""/>
 <part name="SUPPLY2" library="rickk2" deviceset="3V3" device=""/>
@@
 <attribute name="VALUE" x="170.18" y="-78.74" size="1.778" layer="96"/>
 </instance>
-<instance part="SUPPLY4" gate="G$1" x="104.14" y="147.32" smashed="yes">
-<attribute name="VALUE" x="103.124" y="150.876" size="1.778" layer="96"/>
-</instance>
 <instance part="SUPPLY1" gate="G$1" x="66.04" y="144.78" smashed="yes">
