File: src/assets/files/app-notes/AN001/eagle/SomTest1.brd (EAGLE design)
At the start: 31.1 x 85.6 mm, 43 parts, among them U1 MAX17043, U2 BQ24195, U3 XCL223

Commit message: Fix M.2 example
M.2 pin 40 should be D3 and M.2 pin 42 should be D2. These were reversed previously, however
this sample board does not use the pins.
Parts:
- J1: value (none) -> SPARK_M.2EKEY
Other:
- board text added: "SomTest1 v5"
- board text removed: "SomTest1 v4"
Changed lines of the file:
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@@
 <?xml version="1.0" encoding="utf-8"?>
 <!DOCTYPE eagle SYSTEM "eagle.dtd">
-<eagle version="9.4.0">
+<eagle version="9.6.2">
 <drawing>
 <settings>
-<setting alwaysvectorfont="yes"/>
+<setting alwaysvectorfont="no"/>
 <setting verticaltext="up"/>
 </settings>
@@
 <layer number="1" name="Top" color="4" fill="1" visible="yes" active="yes"/>
 <layer number="2" name="Route2" color="16" fill="1" visible="no" active="no"/>
+<layer number="3" name="Route3" color="17" fill="1" visible="no" active="no"/>
+<layer number="4" name="Route4" color="18" fill="1" visible="no" active="no"/>
+<layer number="5" name="Route5" color="19" fill="1" visible="no" active="no"/>
+<layer number="6" name="Route6" color="25" fill="1" visible="no" active="no"/>
+<layer number="7" name="Route7" color="26" fill="1" visible="no" active="no"/>
+<layer number="8" name="Route8" color="27" fill="1" visible="no" active="no"/>
+<layer number="9" name="Route9" color="28" fill="1" visible="no" active="no"/>
+<layer number="10" name="Route10" color="29" fill="1" visible="no" active="no"/>
+<layer number="11" name="Route11" color="30" fill="1" visible="no" active="no"/>
+<layer number="12" name="Route12" color="20" fill="1" visible="no" active="no"/>
+<layer number="13" name="Route13" color="21" fill="1" visible="no" active="no"/>
+<layer number="14" name="Route14" color="22" fill="1" visible="no" active="no"/>
 <layer number="15" name="Route15" color="23" fill="1" visible="no" active="no"/>
 <layer number="16" name="Bottom" color="1" fill="1" visible="yes" active="yes"/>
@@
 <text x="17.145" y="24.765" size="1.27" layer="21" rot="R90">MODE</text>
 <text x="19.05" y="46.99" size="1.27" layer="22" rot="MR0">SomTest1
-v4</text>
+v5</text>
 <text x="6.858" y="6.604" size="0.8128" layer="21">+</text>
 <text x="6.858" y="4.064" size="0.8128" layer="21">-</text>
@@
 <attribute name="NAME" x="4.6228" y="24.1554" size="0.6096" layer="48" rot="R90"/>
 </element>
-<element name="J1" library="rickk2" package="SPARK_M.2EKEY-LESS-CREAM" value="" x="15.24" y="39.37" smashed="yes" rot="R180">
+<element name="J1" library="rickk2" package="SPARK_M.2EKEY-LESS-CREAM" value="SPARK_M.2EKEY" x="15.24" y="39.37" smashed="yes" rot="R180">
 <attribute name="NAME" x="25.2112" y="33.2632" size="1.27" layer="51" rot="R180"/>
 <attribute name="VALUE" x="15.0512" y="33.2632" size="1.27" layer="51" rot="R180"/>
